Commit message: Move go2 models in go2/ subdir

File: model/go2/go2.urdf (robot description, URDF)
Before this commit: robot go2_description, 31 links, 30 joints
Links:
- link FL_calf: geometry collision mesh filename=package://go2_description/model/go2/assets/collisions/calf_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; collision mesh filename=package://go2_description/model/go2/assets/collisions/calf_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
- link FL_foot: geometry collision mesh filename=package://go2_description/model/go2/assets/collisions/foot_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; visual mesh filename=package://go2_description/model/go2/assets/visuals/foot.dae
- link FL_hip: geometry visual mesh filename=package://go2_description/model/go2/assets/visuals/hip.dae
- link FL_thigh: geometry collision mesh filename=package://go2_description/model/go2/assets/collisions/thigh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; visual mesh filename=package://go2_description/model/go2/assets/visuals/thigh.dae
- link FR_calf: geometry collision mesh filename=package://go2_description/model/go2/assets/collisions/calf_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; collision mesh filename=package://go2_description/model/go2/assets/collisions/calf_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
- link FR_foot: geometry collision mesh filename=package://go2_description/model/go2/assets/collisions/foot_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; visual mesh filename=package://go2_description/model/go2/assets/visuals/foot.dae
- link FR_hip: geometry visual mesh filename=package://go2_description/model/go2/assets/visuals/hip.dae
- link FR_thigh: geometry collision mesh filename=package://go2_description/model/go2/assets/collisions/thigh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; visual mesh filename=package://go2_description/model/go2/assets/visuals/thigh_mi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
- link RL_calf: geometry collision mesh filename=package://go2_description/model/go2/assets/collisions/calf_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; collision mesh filename=package://go2_description/model/go2/assets/collisions/calf_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
- link RL_foot: geometry collision mesh filename=package://go2_description/model/go2/assets/collisions/foot_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; visual mesh filename=package://go2_description/model/go2/assets/visuals/foot.dae
- link RL_hip: geometry collision mesh filename=package://go2_description/model/go2/assets/collisions/hip_c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; visual mesh filename=package://go2_description/model/go2/assets/visuals/hip.dae
- link RL_thigh: geometry collision mesh filename=package://go2_description/model/go2/assets/collisions/thigh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; visual mesh filename=package://go2_description/model/go2/assets/visuals/thigh.dae
- link RR_calf: geometry collision mesh filename=package://go2_description/model/go2/assets/collisions/calf_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; collision mesh filename=package://go2_description/model/go2/assets/collisions/calf_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
- link RR_foot: geometry collision mesh filename=package://go2_description/model/go2/assets/collisions/foot_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; visual mesh filename=package://go2_description/model/go2/assets/visuals/foot.dae
- link RR_hip: geometry collision mesh filename=package://go2_description/model/go2/assets/collisions/hip_c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; visual mesh filename=package://go2_description/model/go2/assets/visuals/hip.dae
- link RR_thigh: geometry collision mesh filename=package://go2_description/model/go2/assets/collisions/thigh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; visual mesh filename=package://go2_description/model/go2/assets/visuals/thigh_mi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
- link base: geometry collision mesh filename=package://go2_description/model/go2/assets/collisions/base_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; visual mesh filename=package://go2_description/model/go2/assets/visuals/base.dae
