Commit message: Rename and move files + create loader and path variables

File: model/g1/g1.urdf (robot description, URDF)
Before this commit: robot g1_29dof_lock_waist_rev_1_0, 39 links, 38 joints
Links:
- link head_link: geometry collision mesh filename=package://go2_description/model/g1/assets/head_link.STL; visual mesh filename=package://go2_description/model/g1/assets/head_link.STL
- link left_ankle_pitch_link: geometry collision mesh filename=package://go2_description/model/g1/assets/left_ankle_pitch_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; visual mesh filename=package://go2_description/model/g1/assets/left_ankle_pitch_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
- link left_ankle_roll_link: geometry collision sphere radius=0.005; collision sphere radius=0.005
- link left_elbow_link: geometry collision mesh filename=package://go2_description/model/g1/assets/left_elbow_link.S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; visual mesh filename=package://go2_description/model/g1/assets/left_elbow_link.S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
- link left_hip_pitch_link: geometry collision mesh filename=package://go2_description/model/g1/assets/left_hip_pitch_li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; visual mesh filename=package://go2_description/model/g1/assets/left_hip_pitch_li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
- link left_hip_roll_link: geometry collision mesh filename=package://go2_description/model/g1/assets/left_hip_roll_lin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; visual mesh filename=package://go2_description/model/g1/assets/left_hip_roll_lin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
- link left_hip_yaw_link: geometry collision mesh filename=package://go2_description/model/g1/assets/left_hip_yaw_link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; visual mesh filename=package://go2_description/model/g1/assets/left_hip_yaw_link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
- link left_knee_link: geometry collision mesh filename=package://go2_description/model/g1/assets/left_knee_link.STL; visual mesh filename=package://go2_description/model/g1/assets/left_knee_link.STL
- link left_rubber_hand: geometry visual mesh filename=package://go2_description/model/g1/assets/left_rubber_hand.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
- link left_shoulder_pitch_link: geometry collision cylinder length=0.05 radius=0.03; visual mesh filename=package://go2_description/model/g1/assets/left_shoulder_pit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
- link left_shoulder_roll_link: geometry collision cylinder length=0.03 radius=0.03; visual mesh filename=package://go2_description/model/g1/assets/left_shoulder_rol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
- link left_shoulder_yaw_link: geometry collision mesh filename=package://go2_description/model/g1/assets/left_shoulder_yaw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; visual mesh filename=package://go2_description/model/g1/assets/left_shoulder_yaw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
- link left_wrist_pitch_link: geometry collision mesh filename=package://go2_description/model/g1/assets/left_wrist_pitch_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; visual mesh filename=package://go2_description/model/g1/assets/left_wrist_pitch_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
- link left_wrist_roll_link: geometry collision mesh filename=package://go2_description/model/g1/assets/left_wrist_roll_l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; visual mesh filename=package://go2_description/model/g1/assets/left_wrist_roll_l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
- link left_wrist_yaw_link: geometry collision mesh filename=package://go2_description/model/g1/assets/left_wrist_yaw_li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; visual mesh filename=package://go2_description/model/g1/assets/left_wrist_yaw_li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
- link logo_link: geometry collision mesh filename=package://go2_description/model/g1/assets/logo_link.STL; visual mesh filename=package://go2_description/model/g1/assets/logo_link.STL
- link pelvis: geometry visual mesh filename=package://go2_description/model/g1/assets/pelvis.STL
- link pelvis_contour_link: geometry collision mesh filename=package://go2_description/model/g1/assets/pelvis_contour_li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; visual mesh filename=package://go2_description/model/g1/assets/pelvis_contour_li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
- link right_ankle_pitch_link: geometry collision mesh filename=package://go2_description/model/g1/assets/right_ankle_pitch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; visual mesh filename=package://go2_description/model/g1/assets/right_ankle_pitch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
- link right_ankle_roll_link: geometry collision sphere radius=0.005; collision sphere radius=0.005
- link right_elbow_link: geometry collision mesh filename=package://go2_description/model/g1/assets/right_elbow_link.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; visual mesh filename=package://go2_description/model/g1/assets/right_elbow_link.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
- link right_hip_pitch_link: geometry collision mesh filename=package://go2_description/model/g1/assets/right_hip_pitch_l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; visual mesh filename=package://go2_description/model/g1/assets/right_hip_pitch_l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
- link right_hip_roll_link: geometry collision mesh filename=package://go2_description/model/g1/assets/right_hip_roll_li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; visual mesh filename=package://go2_description/model/g1/assets/right_hip_roll_li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
- link right_hip_yaw_link: geometry collision mesh filename=package://go2_description/model/g1/assets/right_hip_yaw_lin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; visual mesh filename=package://go2_description/model/g1/assets/right_hip_yaw_lin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
- link right_knee_link: geometry collision mesh filename=package://go2_description/model/g1/assets/right_knee_link.S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; visual mesh filename=package://go2_description/model/g1/assets/right_knee_link.S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
- link right_rubber_hand: geometry visual mesh filename=package://go2_description/model/g1/assets/right_rubber_hand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
- link right_shoulder_pitch_link: geometry collision cylinder length=0.05 radius=0.03; visual mesh filename=package://go2_description/model/g1/assets/right_shoulder_pi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
- link right_shoulder_roll_link: geometry collision cylinder length=0.03 radius=0.03; visual mesh filename=package://go2_description/model/g1/assets/right_shoulder_ro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
- link right_shoulder_yaw_link: geometry collision mesh filename=package://go2_description/model/g1/assets/right_shoulder_ya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; visual mesh filename=package://go2_description/model/g1/assets/right_shoulder_ya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
- link right_wrist_pitch_link: geometry collision mesh filename=package://go2_description/model/g1/assets/right_wrist_pitch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; visual mesh filename=package://go2_description/model/g1/assets/right_wrist_pitch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
- link right_wrist_roll_link: geometry collision mesh filename=package://go2_description/model/g1/assets/right_wrist_roll_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; visual mesh filename=package://go2_description/model/g1/assets/right_wrist_roll_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
- link right_wrist_yaw_link: geometry collision mesh filename=package://go2_description/model/g1/assets/right_wrist_yaw_l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; visual mesh filename=package://go2_description/model/g1/assets/right_wrist_yaw_l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
- link torso_link: geometry collision mesh filename=package://go2_description/model/g1/assets/torso_link_rev_1_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; visual mesh filename=package://go2_description/model/g1/assets/torso_link_rev_1_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
- link waist_roll_link: geometry visual mesh filename=package://go2_description/model/g1/assets/waist_roll_link_r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
- link waist_yaw_link: geometry visual mesh filename=package://go2_description/model/g1/assets/waist_yaw_link_re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

Commit message: Remove collisions

File: model/g1/g1.urdf (robot description, URDF)
Before this commit: robot g1_29dof_lock_waist_rev_1_0, 39 links, 38 joints
Links:
- link head_link: geometry visual mesh filename=package://go2_description/model/g1/assets/head_link.STL
- link left_ankle_pitch_link: geometry visual mesh filename=package://go2_description/model/g1/assets/left_ankle_pitch_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
- link left_ankle_roll_link: geometry visual mesh filename=package://go2_description/model/g1/assets/left_ankle_roll_l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
- link left_elbow_link: geometry visual mesh filename=package://go2_description/model/g1/assets/left_elbow_link.S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
- link left_hip_pitch_link: geometry visual mesh filename=package://go2_description/model/g1/assets/left_hip_pitch_li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
- link left_hip_roll_link: geometry visual mesh filename=package://go2_description/model/g1/assets/left_hip_roll_lin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
- link left_hip_yaw_link: geometry visual mesh filename=package://go2_description/model/g1/assets/left_hip_yaw_link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
- link left_knee_link: geometry visual mesh filename=package://go2_description/model/g1/assets/left_knee_link.STL
- link left_shoulder_pitch_link: geometry visual mesh filename=package://go2_description/model/g1/assets/left_shoulder_pit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
- link left_shoulder_roll_link: geometry visual mesh filename=package://go2_description/model/g1/assets/left_shoulder_rol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
- link left_shoulder_yaw_link: geometry visual mesh filename=package://go2_description/model/g1/assets/left_shoulder_yaw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
- link left_wrist_pitch_link: geometry visual mesh filename=package://go2_description/model/g1/assets/left_wrist_pitch_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
- link left_wrist_roll_link: geometry visual mesh filename=package://go2_description/model/g1/assets/left_wrist_roll_l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
- link left_wrist_yaw_link: geometry visual mesh filename=package://go2_description/model/g1/assets/left_wrist_yaw_li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
- link logo_link: geometry visual mesh filename=package://go2_description/model/g1/assets/logo_link.STL
- link pelvis_contour_link: geometry visual mesh filename=package://go2_description/model/g1/assets/pelvis_contour_li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
- link right_ankle_pitch_link: geometry visual mesh filename=package://go2_description/model/g1/assets/right_ankle_pitch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
- link right_ankle_roll_link: geometry visual mesh filename=package://go2_description/model/g1/assets/right_ankle_roll_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
- link right_elbow_link: geometry visual mesh filename=package://go2_description/model/g1/assets/right_elbow_link.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
- link right_hip_pitch_link: geometry visual mesh filename=package://go2_description/model/g1/assets/right_hip_pitch_l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
- link right_hip_roll_link: geometry visual mesh filename=package://go2_description/model/g1/assets/right_hip_roll_li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
- link right_hip_yaw_link: geometry visual mesh filename=package://go2_description/model/g1/assets/right_hip_yaw_lin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
- link right_knee_link: geometry visual mesh filename=package://go2_description/model/g1/assets/right_knee_link.S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
- link right_shoulder_pitch_link: geometry visual mesh filename=package://go2_description/model/g1/assets/right_shoulder_pi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
- link right_shoulder_roll_link: geometry visual mesh filename=package://go2_description/model/g1/assets/right_shoulder_ro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
- link right_shoulder_yaw_link: geometry visual mesh filename=package://go2_description/model/g1/assets/right_shoulder_ya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
- link right_wrist_pitch_link: geometry visual mesh filename=package://go2_description/model/g1/assets/right_wrist_pitch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
- link right_wrist_roll_link: geometry visual mesh filename=package://go2_description/model/g1/assets/right_wrist_roll_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
- link right_wrist_yaw_link: geometry visual mesh filename=package://go2_description/model/g1/assets/right_wrist_yaw_l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
- link torso_link: geometry visual mesh filename=package://go2_description/model/g1/assets/torso_link_rev_1_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

Commit message: Duplicate visual models to collisions and remove origin when zero

File: model/g1/g1.urdf (robot description, URDF)
Before this commit: robot g1_29dof_lock_waist_rev_1_0, 39 links, 38 joints
Links:
- link head_link: geometry collision mesh filename=package://go2_description/model/g1/assets/collision/head_li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; visual mesh filename=package://go2_description/model/g1/assets/head_link.STL
- link left_ankle_pitch_link: geometry collision mesh filename=package://go2_description/model/g1/assets/collision/left_an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; visual mesh filename=package://go2_description/model/g1/assets/left_ankle_pitch_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
- link left_ankle_roll_link: geometry collision mesh filename=package://go2_description/model/g1/assets/collision/left_an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; visual mesh filename=package://go2_description/model/g1/assets/left_ankle_roll_l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
- link left_elbow_link: geometry collision mesh filename=package://go2_description/model/g1/assets/collision/left_el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; visual mesh filename=package://go2_description/model/g1/assets/left_elbow_link.S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
- link left_hip_pitch_link: geometry collision mesh filename=package://go2_description/model/g1/assets/collision/left_hi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; visual mesh filename=package://go2_description/model/g1/assets/left_hip_pitch_li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
- link left_hip_roll_link: geometry collision mesh filename=package://go2_description/model/g1/assets/collision/left_hi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; visual mesh filename=package://go2_description/model/g1/assets/left_hip_roll_lin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
- link left_hip_yaw_link: geometry collision mesh filename=package://go2_description/model/g1/assets/collision/left_hi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; visual mesh filename=package://go2_description/model/g1/assets/left_hip_yaw_link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
- link left_knee_link: geometry collision mesh filename=package://go2_description/model/g1/assets/collision/left_kn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; visual mesh filename=package://go2_description/model/g1/assets/left_knee_link.STL
- link left_rubber_hand: geometry collision mesh filename=package://go2_description/model/g1/assets/collision/left_ru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; visual mesh filename=package://go2_description/model/g1/assets/left_rubber_hand.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
- link left_shoulder_pitch_link: geometry collision mesh filename=package://go2_description/model/g1/assets/collision/left_sh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; visual mesh filename=package://go2_description/model/g1/assets/left_shoulder_pit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
- link left_shoulder_roll_link: geometry collision mesh filename=package://go2_description/model/g1/assets/collision/left_sh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; visual mesh filename=package://go2_description/model/g1/assets/left_shoulder_rol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
- link left_shoulder_yaw_link: geometry collision mesh filename=package://go2_description/model/g1/assets/collision/left_sh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; visual mesh filename=package://go2_description/model/g1/assets/left_shoulder_yaw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
- link left_wrist_pitch_link: geometry collision mesh filename=package://go2_description/model/g1/assets/collision/left_wr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; visual mesh filename=package://go2_description/model/g1/assets/left_wrist_pitch_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
- link left_wrist_roll_link: geometry collision mesh filename=package://go2_description/model/g1/assets/collision/left_wr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; visual mesh filename=package://go2_description/model/g1/assets/left_wrist_roll_l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
- link left_wrist_yaw_link: geometry collision mesh filename=package://go2_description/model/g1/assets/collision/left_wr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; visual mesh filename=package://go2_description/model/g1/assets/left_wrist_yaw_li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
- link logo_link: geometry collision mesh filename=package://go2_description/model/g1/assets/collision/logo_li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; visual mesh filename=package://go2_description/model/g1/assets/logo_link.STL
- link pelvis: geometry collision mesh filename=package://go2_description/model/g1/assets/collision/pelvis_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; visual mesh filename=package://go2_description/model/g1/assets/pelvis.STL
- link pelvis_contour_link: geometry collision mesh filename=package://go2_description/model/g1/assets/collision/pelvis_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; visual mesh filename=package://go2_description/model/g1/assets/pelvis_contour_li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
- link right_ankle_pitch_link: geometry collision mesh filename=package://go2_description/model/g1/assets/collision/right_a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; visual mesh filename=package://go2_description/model/g1/assets/right_ankle_pitch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
- link right_ankle_roll_link: geometry collision mesh filename=package://go2_description/model/g1/assets/collision/right_a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; visual mesh filename=package://go2_description/model/g1/assets/right_ankle_roll_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
- link right_elbow_link: geometry collision mesh filename=package://go2_description/model/g1/assets/collision/right_e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; visual mesh filename=package://go2_description/model/g1/assets/right_elbow_link.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
- link right_hip_pitch_link: geometry collision mesh filename=package://go2_description/model/g1/assets/collision/right_h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; visual mesh filename=package://go2_description/model/g1/assets/right_hip_pitch_l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
- link right_hip_roll_link: geometry collision mesh filename=package://go2_description/model/g1/assets/collision/right_h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; visual mesh filename=package://go2_description/model/g1/assets/right_hip_roll_li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
- link right_hip_yaw_link: geometry collision mesh filename=package://go2_description/model/g1/assets/collision/right_h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; visual mesh filename=package://go2_description/model/g1/assets/right_hip_yaw_lin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
- link right_knee_link: geometry collision mesh filename=package://go2_description/model/g1/assets/collision/right_k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; visual mesh filename=package://go2_description/model/g1/assets/right_knee_link.S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
- link right_rubber_hand: geometry collision mesh filename=package://go2_description/model/g1/assets/collision/right_r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; visual mesh filename=package://go2_description/model/g1/assets/right_rubber_hand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
- link right_shoulder_pitch_link: geometry collision mesh filename=package://go2_description/model/g1/assets/collision/right_s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; visual mesh filename=package://go2_description/model/g1/assets/right_shoulder_pi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
- link right_shoulder_roll_link: geometry collision mesh filename=package://go2_description/model/g1/assets/collision/right_s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; visual mesh filename=package://go2_description/model/g1/assets/right_shoulder_ro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
- link right_shoulder_yaw_link: geometry collision mesh filename=package://go2_description/model/g1/assets/collision/right_s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; visual mesh filename=package://go2_description/model/g1/assets/right_shoulder_ya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
- link right_wrist_pitch_link: geometry collision mesh filename=package://go2_description/model/g1/assets/collision/right_w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; visual mesh filename=package://go2_description/model/g1/assets/right_wrist_pitch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
- link right_wrist_roll_link: geometry collision mesh filename=package://go2_description/model/g1/assets/collision/right_w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; visual mesh filename=package://go2_description/model/g1/assets/right_wrist_roll_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
- link right_wrist_yaw_link: geometry collision mesh filename=package://go2_description/model/g1/assets/collision/right_w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; visual mesh filename=package://go2_description/model/g1/assets/right_wrist_yaw_l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
- link torso_link: geometry collision mesh filename=package://go2_description/model/g1/assets/collision/torso_l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; visual mesh filename=package://go2_description/model/g1/assets/torso_link_rev_1_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
- link waist_roll_link: geometry collision mesh filename=package://go2_description/model/g1/assets/collision/waist_r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; visual mesh filename=package://go2_description/model/g1/assets/waist_roll_link_r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
- link waist_yaw_link: geometry collision mesh filename=package://go2_description/model/g1/assets/collision/waist_y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; visual mesh filename=package://go2_description/model/g1/assets/waist_yaw_link_re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
Joints:
- joint waist_pitch_joint: origin xyz=0 0 0 rpy=0 0 0 -> (none)
- joint waist_yaw_joint: origin xyz=0 0 0 rpy=0 0 0 -> (none)
