Commit message: Move mesh to visuals

File: model/g1/g1.urdf (robot description, URDF)
Before this commit: robot g1_29dof_lock_waist_rev_1_0, 39 links, 38 joints
Links:
- link head_link: geometry collision mesh filename=package://go2_description/model/g1/assets/collisions/head_l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; visual mesh filename=package://go2_description/model/g1/assets/visuals/head_link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
- link left_ankle_pitch_link: geometry collision mesh filename=package://go2_description/model/g1/assets/collisions/left_a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; visual mesh filename=package://go2_description/model/g1/assets/visuals/left_ankl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
- link left_ankle_roll_link: geometry collision mesh filename=package://go2_description/model/g1/assets/collisions/left_a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; visual mesh filename=package://go2_description/model/g1/assets/visuals/left_ankl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
- link left_elbow_link: geometry collision mesh filename=package://go2_description/model/g1/assets/collisions/left_e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; visual mesh filename=package://go2_description/model/g1/assets/visuals/left_elbo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
- link left_hip_pitch_link: geometry collision mesh filename=package://go2_description/model/g1/assets/collisions/left_h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; visual mesh filename=package://go2_description/model/g1/assets/visuals/left_hip_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
- link left_hip_roll_link: geometry collision mesh filename=package://go2_description/model/g1/assets/collisions/left_h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; visual mesh filename=package://go2_description/model/g1/assets/visuals/left_hip_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
- link left_hip_yaw_link: geometry collision mesh filename=package://go2_description/model/g1/assets/collisions/left_h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; visual mesh filename=package://go2_description/model/g1/assets/visuals/left_hip_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
- link left_knee_link: geometry collision mesh filename=package://go2_description/model/g1/assets/collisions/left_k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; visual mesh filename=package://go2_description/model/g1/assets/visuals/left_knee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
- link left_rubber_hand: geometry collision mesh filename=package://go2_description/model/g1/assets/collisions/left_r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; visual mesh filename=package://go2_description/model/g1/assets/visuals/left_rubb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
- link left_shoulder_pitch_link: geometry collision mesh filename=package://go2_description/model/g1/assets/collisions/left_s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; visual mesh filename=package://go2_description/model/g1/assets/visuals/left_shou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
- link left_shoulder_roll_link: geometry collision mesh filename=package://go2_description/model/g1/assets/collisions/left_s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; visual mesh filename=package://go2_description/model/g1/assets/visuals/left_shou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
- link left_shoulder_yaw_link: geometry collision mesh filename=package://go2_description/model/g1/assets/collisions/left_s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; visual mesh filename=package://go2_description/model/g1/assets/visuals/left_shou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
- link left_wrist_pitch_link: geometry collision mesh filename=package://go2_description/model/g1/assets/collisions/left_w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; visual mesh filename=package://go2_description/model/g1/assets/visuals/left_wris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
- link left_wrist_roll_link: geometry collision mesh filename=package://go2_description/model/g1/assets/collisions/left_w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; visual mesh filename=package://go2_description/model/g1/assets/visuals/left_wris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
- link left_wrist_yaw_link: geometry collision mesh filename=package://go2_description/model/g1/assets/collisions/left_w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; visual mesh filename=package://go2_description/model/g1/assets/visuals/left_wris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
- link logo_link: geometry collision mesh filename=package://go2_description/model/g1/assets/collisions/logo_l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; visual mesh filename=package://go2_description/model/g1/assets/visuals/logo_link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
- link pelvis: geometry collision mesh filename=package://go2_description/model/g1/assets/collisions/pelvis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; visual mesh filename=package://go2_description/model/g1/assets/visuals/pelvis.STL
- link pelvis_contour_link: geometry collision mesh filename=package://go2_description/model/g1/assets/collisions/pelvis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; visual mesh filename=package://go2_description/model/g1/assets/visuals/pelvis_co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
- link right_ankle_pitch_link: geometry collision mesh filename=package://go2_description/model/g1/assets/collisions/right_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; visual mesh filename=package://go2_description/model/g1/assets/visuals/right_ank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
- link right_ankle_roll_link: geometry collision mesh filename=package://go2_description/model/g1/assets/collisions/right_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; visual mesh filename=package://go2_description/model/g1/assets/visuals/right_ank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
- link right_elbow_link: geometry collision mesh filename=package://go2_description/model/g1/assets/collisions/right_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; visual mesh filename=package://go2_description/model/g1/assets/visuals/right_elb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
- link right_hip_pitch_link: geometry collision mesh filename=package://go2_description/model/g1/assets/collisions/right_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; visual mesh filename=package://go2_description/model/g1/assets/visuals/right_hip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
- link right_hip_roll_link: geometry collision mesh filename=package://go2_description/model/g1/assets/collisions/right_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; visual mesh filename=package://go2_description/model/g1/assets/visuals/right_hip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
- link right_hip_yaw_link: geometry collision mesh filename=package://go2_description/model/g1/assets/collisions/right_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; visual mesh filename=package://go2_description/model/g1/assets/visuals/right_hip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
- link right_knee_link: geometry collision mesh filename=package://go2_description/model/g1/assets/collisions/right_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; visual mesh filename=package://go2_description/model/g1/assets/visuals/right_kne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
- link right_rubber_hand: geometry collision mesh filename=package://go2_description/model/g1/assets/collisions/right_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; visual mesh filename=package://go2_description/model/g1/assets/visuals/right_rub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
- link right_shoulder_pitch_link: geometry collision mesh filename=package://go2_description/model/g1/assets/collisions/right_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; visual mesh filename=package://go2_description/model/g1/assets/visuals/right_sho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
- link right_shoulder_roll_link: geometry collision mesh filename=package://go2_description/model/g1/assets/collisions/right_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; visual mesh filename=package://go2_description/model/g1/assets/visuals/right_sho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
- link right_shoulder_yaw_link: geometry collision mesh filename=package://go2_description/model/g1/assets/collisions/right_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; visual mesh filename=package://go2_description/model/g1/assets/visuals/right_sho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
- link right_wrist_pitch_link: geometry collision mesh filename=package://go2_description/model/g1/assets/collisions/right_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; visual mesh filename=package://go2_description/model/g1/assets/visuals/right_wri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
- link right_wrist_roll_link: geometry collision mesh filename=package://go2_description/model/g1/assets/collisions/right_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; visual mesh filename=package://go2_description/model/g1/assets/visuals/right_wri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
- link right_wrist_yaw_link: geometry collision mesh filename=package://go2_description/model/g1/assets/collisions/right_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; visual mesh filename=package://go2_description/model/g1/assets/visuals/right_wri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
- link torso_link: geometry collision mesh filename=package://go2_description/model/g1/assets/collisions/torso_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; visual mesh filename=package://go2_description/model/g1/assets/visuals/torso_lin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
- link waist_roll_link: geometry collision mesh filename=package://go2_description/model/g1/assets/collisions/waist_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; visual mesh filename=package://go2_description/model/g1/assets/visuals/waist_rol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
- link waist_yaw_link: geometry collision mesh filename=package://go2_description/model/g1/assets/collisions/waist_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; visual mesh filename=package://go2_description/model/g1/assets/visuals/waist_yaw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

Commit message: Remove logo collision

File: model/g1/g1.urdf (robot description, URDF)
Before this commit: robot g1_29dof_lock_waist_rev_1_0, 39 links, 38 joints
Links:
- link logo_link: geometry visual mesh filename=package://go2_description/model/g1/assets/visuals/logo_link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

Commit message: Merge wrist and hand collision to reduce pairs

File: model/g1/g1.urdf (robot description, URDF)
Before this commit: robot g1, 39 links, 38 joints
Links:
- link left_rubber_hand: geometry collision mesh filename=package://go2_description/model/g1/assets/collisions/left_w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; visual mesh filename=package://go2_description/model/g1/assets/visuals/left_rubb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
- link left_wrist_yaw_link: geometry visual mesh filename=package://go2_description/model/g1/assets/visuals/left_wris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
- link right_wrist_yaw_link: geometry visual mesh filename=package://go2_description/model/g1/assets/visuals/right_wri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

Commit message: Merge pelvis collisions

File: model/g1/g1.urdf (robot description, URDF)
Before this commit: robot g1, 39 links, 38 joints
Links:
- link pelvis_contour_link: geometry visual mesh filename=package://go2_description/model/g1/assets/visuals/pelvis_co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

Commit message: Merge torso and waist collision link (since fixed waist for now)

File: model/g1/g1.urdf (robot description, URDF)
Before this commit: robot g1, 39 links, 38 joints
Links:
- link waist_roll_link: geometry visual mesh filename=package://go2_description/model/g1/assets/visuals/waist_rol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
- link waist_yaw_link: geometry visual mesh filename=package://go2_description/model/g1/assets/visuals/waist_yaw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

Commit message: Remove useless ankle pitch link collision

File: model/g1/g1.urdf (robot description, URDF)
Before this commit: robot g1, 39 links, 38 joints
Links:
- link left_ankle_pitch_link: geometry visual mesh filename=package://go2_description/model/g1/assets/visuals/left_ankl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
- link right_ankle_pitch_link: geometry visual mesh filename=package://go2_description/model/g1/assets/visuals/right_ank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

Commit message: Add battery mass and inertia

File: model/g1/g1.urdf (robot description, URDF)
Before this commit: robot g1, 39 links, 38 joints
Links:
- added link battery, mass 2.5
Joints:
- added joint battery_joint: type fixed, parent imu_in_torso, child battery, origin xyz=0.05 0.025 -0.01 rpy=0 0 0

Commit message: Rename to unitree_description

File: model/g1/g1.urdf (robot description, URDF)
Before this commit: robot g1, 40 links, 39 joints
Links:
- link head_link: geometry collision mesh filename=package://unitree_description/model/g1/assets/collisions/he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; visual mesh filename=package://unitree_description/model/g1/assets/visuals/head_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
- link left_ankle_pitch_link: geometry visual mesh filename=package://unitree_description/model/g1/assets/visuals/left_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
- link left_ankle_roll_link: geometry collision mesh filename=package://unitree_description/model/g1/assets/collisions/le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; visual mesh filename=package://unitree_description/model/g1/assets/visuals/left_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
- link left_elbow_link: geometry collision mesh filename=package://unitree_description/model/g1/assets/collisions/le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; visual mesh filename=package://unitree_description/model/g1/assets/visuals/left_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
- link left_hip_pitch_link: geometry collision mesh filename=package://unitree_description/model/g1/assets/collisions/le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; visual mesh filename=package://unitree_description/model/g1/assets/visuals/left_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
- link left_hip_roll_link: geometry collision mesh filename=package://unitree_description/model/g1/assets/collisions/le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; visual mesh filename=package://unitree_description/model/g1/assets/visuals/left_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
- link left_hip_yaw_link: geometry collision mesh filename=package://unitree_description/model/g1/assets/collisions/le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; visual mesh filename=package://unitree_description/model/g1/assets/visuals/left_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
- link left_knee_link: geometry collision mesh filename=package://unitree_description/model/g1/assets/collisions/le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; visual mesh filename=package://unitree_description/model/g1/assets/visuals/left_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
- link left_rubber_hand: geometry collision mesh filename=package://unitree_description/model/g1/assets/collisions/le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; visual mesh filename=package://unitree_description/model/g1/assets/visuals/left_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
- link left_shoulder_pitch_link: geometry collision mesh filename=package://unitree_description/model/g1/assets/collisions/le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; visual mesh filename=package://unitree_description/model/g1/assets/visuals/left_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
- link left_shoulder_roll_link: geometry collision mesh filename=package://unitree_description/model/g1/assets/collisions/le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; visual mesh filename=package://unitree_description/model/g1/assets/visuals/left_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
- link left_shoulder_yaw_link: geometry collision mesh filename=package://unitree_description/model/g1/assets/collisions/le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; visual mesh filename=package://unitree_description/model/g1/assets/visuals/left_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
- link left_wrist_pitch_link: geometry collision mesh filename=package://unitree_description/model/g1/assets/collisions/le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; visual mesh filename=package://unitree_description/model/g1/assets/visuals/left_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
- link left_wrist_roll_link: geometry collision mesh filename=package://unitree_description/model/g1/assets/collisions/le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; visual mesh filename=package://unitree_description/model/g1/assets/visuals/left_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
- link left_wrist_yaw_link: geometry visual mesh filename=package://unitree_description/model/g1/assets/visuals/left_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
- link logo_link: geometry visual mesh filename=package://unitree_description/model/g1/assets/visuals/logo_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
- link pelvis: geometry collision mesh filename=package://unitree_description/model/g1/assets/collisions/pe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; visual mesh filename=package://unitree_description/model/g1/assets/visuals/pelvi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
- link pelvis_contour_link: geometry visual mesh filename=package://unitree_description/model/g1/assets/visuals/pelvi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
- link right_ankle_pitch_link: geometry visual mesh filename=package://unitree_description/model/g1/assets/visuals/right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
- link right_ankle_roll_link: geometry collision mesh filename=package://unitree_description/model/g1/assets/collisions/ri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; visual mesh filename=package://unitree_description/model/g1/assets/visuals/right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
- link right_elbow_link: geometry collision mesh filename=package://unitree_description/model/g1/assets/collisions/ri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; visual mesh filename=package://unitree_description/model/g1/assets/visuals/right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
- link right_hip_pitch_link: geometry collision mesh filename=package://unitree_description/model/g1/assets/collisions/ri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; visual mesh filename=package://unitree_description/model/g1/assets/visuals/right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
- link right_hip_roll_link: geometry collision mesh filename=package://unitree_description/model/g1/assets/collisions/ri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; visual mesh filename=package://unitree_description/model/g1/assets/visuals/right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
- link right_hip_yaw_link: geometry collision mesh filename=package://unitree_description/model/g1/assets/collisions/ri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; visual mesh filename=package://unitree_description/model/g1/assets/visuals/right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
- link right_knee_link: geometry collision mesh filename=package://unitree_description/model/g1/assets/collisions/ri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; visual mesh filename=package://unitree_description/model/g1/assets/visuals/right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
- link right_rubber_hand: geometry collision mesh filename=package://unitree_description/model/g1/assets/collisions/ri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; visual mesh filename=package://unitree_description/model/g1/assets/visuals/right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
- link right_shoulder_pitch_link: geometry collision mesh filename=package://unitree_description/model/g1/assets/collisions/ri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; visual mesh filename=package://unitree_description/model/g1/assets/visuals/right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
- link right_shoulder_roll_link: geometry collision mesh filename=package://unitree_description/model/g1/assets/collisions/ri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; visual mesh filename=package://unitree_description/model/g1/assets/visuals/right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
- link right_shoulder_yaw_link: geometry collision mesh filename=package://unitree_description/model/g1/assets/collisions/ri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; visual mesh filename=package://unitree_description/model/g1/assets/visuals/right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
- link right_wrist_pitch_link: geometry collision mesh filename=package://unitree_description/model/g1/assets/collisions/ri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; visual mesh filename=package://unitree_description/model/g1/assets/visuals/right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
- link right_wrist_roll_link: geometry collision mesh filename=package://unitree_description/model/g1/assets/collisions/ri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; visual mesh filename=package://unitree_description/model/g1/assets/visuals/right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
- link right_wrist_yaw_link: geometry visual mesh filename=package://unitree_description/model/g1/assets/visuals/right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
- link torso_link: geometry collision mesh filename=package://unitree_description/model/g1/assets/collisions/to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; visual mesh filename=package://unitree_description/model/g1/assets/visuals/torso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
- link waist_roll_link: geometry visual mesh filename=package://unitree_description/model/g1/assets/visuals/waist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
- link waist_yaw_link: geometry visual mesh filename=package://unitree_description/model/g1/assets/visuals/waist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

File: model/go2/go2.urdf (robot description, URDF)
Before this commit: robot go2_description, 31 links, 30 joints
Links:
- link FL_calf: geometry collision mesh filename=package://unitree_description/model/go2/assets/collisions/c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; collision mesh filename=package://unitree_description/model/go2/assets/collisions/c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
- link FL_foot: geometry collision mesh filename=package://unitree_description/model/go2/assets/collisions/f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; visual mesh filename=package://unitree_description/model/go2/assets/visuals/foot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
- link FL_hip: geometry visual mesh filename=package://unitree_description/model/go2/assets/visuals/hip.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
- link FL_thigh: geometry collision mesh filename=package://unitree_description/model/go2/assets/collisions/t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; visual mesh filename=package://unitree_description/model/go2/assets/visuals/thig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
- link FR_calf: geometry collision mesh filename=package://unitree_description/model/go2/assets/collisions/c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; collision mesh filename=package://unitree_description/model/go2/assets/collisions/c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
- link FR_foot: geometry collision mesh filename=package://unitree_description/model/go2/assets/collisions/f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; visual mesh filename=package://unitree_description/model/go2/assets/visuals/foot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
- link FR_hip: geometry visual mesh filename=package://unitree_description/model/go2/assets/visuals/hip.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
- link FR_thigh: geometry collision mesh filename=package://unitree_description/model/go2/assets/collisions/t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; visual mesh filename=package://unitree_description/model/go2/assets/visuals/thig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
- link RL_calf: geometry collision mesh filename=package://unitree_description/model/go2/assets/collisions/c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; collision mesh filename=package://unitree_description/model/go2/assets/collisions/c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
- link RL_foot: geometry collision mesh filename=package://unitree_description/model/go2/assets/collisions/f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; visual mesh filename=package://unitree_description/model/go2/assets/visuals/foot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
- link RL_hip: geometry collision mesh filename=package://unitree_description/model/go2/assets/collisions/h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; visual mesh filename=package://unitree_description/model/go2/assets/visuals/hip.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
- link RL_thigh: geometry collision mesh filename=package://unitree_description/model/go2/assets/collisions/t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; visual mesh filename=package://unitree_description/model/go2/assets/visuals/thig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
- link RR_calf: geometry collision mesh filename=package://unitree_description/model/go2/assets/collisions/c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; collision mesh filename=package://unitree_description/model/go2/assets/collisions/c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
- link RR_foot: geometry collision mesh filename=package://unitree_description/model/go2/assets/collisions/f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; visual mesh filename=package://unitree_description/model/go2/assets/visuals/foot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
- link RR_hip: geometry collision mesh filename=package://unitree_description/model/go2/assets/collisions/h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; visual mesh filename=package://unitree_description/model/go2/assets/visuals/hip.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
- link RR_thigh: geometry collision mesh filename=package://unitree_description/model/go2/assets/collisions/t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; visual mesh filename=package://unitree_description/model/go2/assets/visuals/thig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
- link base: geometry collision mesh filename=package://unitree_description/model/go2/assets/collisions/b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; visual mesh filename=package://unitree_description/model/go2/assets/visuals/base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
